File: Hardware/Qwiic_IMU_Bonobo.sch (EAGLE design)
At the start: 41 parts, among them J2 SMD, J3 PTH, J4 SMD, J6 SPI, U2 BNO080, Y1 32.768kHz

Commit message: Silk updated to BNO086 and vectors
-Product name silk updated to BNO086
-all silk updated to vector buzzard style
-Jumpers updated to newest packages
Parts:
- removed SJ2: SOLDERJUMPERNO, SparkFun:SOLDERJUMPERNO
- added ADR: JUMPER-SMT_2_NO_SILK, SparkFun-Jumpers:JUMPER-SMT_2_NO_SILK
- SJ3, SJ4: value SOLDERJUMPERNO -> JUMPER-SMT_2_NO_SILK; device SparkFun:SOLDERJUMPERNO -> SparkFun-Jumpers:JUMPER-SMT_2_NO_SILK
Connections:
- net ADDR/MOSI: now also ADR.2; no longer SJ2.2
- net GND: now also ADR.1; no longer SJ2.1

Commit message: minor stuff - measures, library work
-added measures and units
-replaced some connectors, fids, standoffs, GND symbols to newer libraries.
-renamed jumpers (in SCH) to match silk names (on board).
-Red LED to new King Bright version, also updated resistor value to 4.7K
-some minor schematic cleanup
Parts:
- removed D1: RED, SparkFun-LED:LED-RED0603
- added PWR: RED, SparkFun-LED:LED-RED_0603-KB
- J2, J4: device SparkX:I2C_STANDARDJS-1MM -> SparkFun-Connectors:QWIIC_CONNECTORJS-1MM
- J3: device SparkX:I2C_STANDARD_NO_SILK -> SparkFun-Connectors:I2C_STANDARD_NO_SILK
- JP1, JP2, JP5, JP6: device SparkFun:FIDUCIALUFIDUCIAL -> SparkFun-Aesthetics:FIDUCIALUFIDUCIAL
- JP3, JP4: device SparkFun:STAND-OFF -> SparkFun-Hardware:STAND-OFF
- R2: value 1k -> 4.7k; device SparkFun-Resistors:1KOHM-0603-1/10W-1% -> SparkFun-Resistors:4.7KOHM-0603-1/10W-1%
- renumbered SJ1 to I2C, SJ3 to PS0, SJ4 to PS1
Connections:
- net 3.3V: now also J2.2, J3.2, J4.2, PWR.A; no longer D1.A, J2.VCC, J3.VCC, J4.VCC
- net GND: now also J2.1, J3.1, J4.1; no longer J2.GND, J3.GND, J4.GND
- net N$3: now also PWR.C; no longer D1.C
- net SCL/SCK/RX: now also J2.4, J3.4, J4.4; no longer J2.SCL, J3.SCL, J4.SCL
- net SDA/MISO/TX: now also J2.3, J3.3, J4.3; no longer J2.SDA, J3.SDA, J4.SDA
Other:
- note removed: "Power"
- moved on the sheet: C3, C5
